File: PCB/MOSFET.kicad_sch (KiCad schematic)
At the start: 9 parts, among them J6 Conn_02x02_Counter_Clockwise, Q1 BSC026N08NS5, Q2 BSC026N08NS5

Commit message: Updated USB plug, Updated Part Numbers
Parts:
- R3: JLC C2985721 -> C2903495; LCSC C2985721 -> C2903495
Changed lines of the file:
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@@
 			)
 		)
-		(property "LCSC" "C2985721"
+		(property "LCSC" "C2903495"
 			(at 195.58 83.82 0)
 			(effects
@@
 			)
 		)
-		(property "JLC" "C2985721"
+		(property "JLC" "C2903495"
 			(at 195.58 83.82 0)
 			(effects
