File: PCB/Power.kicad_sch (KiCad schematic)
At the start: 20 parts, among them J10 Conn_01x06_Male, J9 Conn_01x06_Male, U1 TMC6200-TA

Commit message: Updated USB plug, Updated Part Numbers
Parts:
- C4, C5: JLC C49217 -> C377773; LCSC C49217 -> C377773
Changed lines of the file:
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@@
 			)
 		)
-		(property "JLC" "C49217"
+		(property "JLC" "C377773"
 			(at 39.37 41.91 0)
 			(effects
@@
 			)
 		)
-		(property "LCSC" "C49217"
+		(property "LCSC" "C377773"
 			(at 39.37 41.91 0)
 			(effects
@@
 			)
 		)
-		(property "JLC" "C49217"
+		(property "JLC" "C377773"
 			(at 46.99 39.37 0)
 			(effects
@@
 			)
 		)
-		(property "LCSC" "C49217"
+		(property "LCSC" "C377773"
 			(at 46.99 39.37 0)
 			(effects
