File: PCB/xESC2.kicad_sch (KiCad schematic)
At the start: 44 parts, among them J1 Conn_01x06_Male, J2 USB_B_Micro, J3 Conn_01x05_Male, J4 Conn_01x05_Male, J5 Conn_01x03_Male, U5 SN65HVD232

Commit message: Updated USB plug, Updated Part Numbers
Parts:
- J2: footprint Connector_USB:USB_Micro-B_Wuerth_614105150721_Vertical -> xESC2:USB_Micro; JLC C668588 -> C145795
Changed lines of the file:
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@@
 			)
 		)
-		(property "Footprint" "Connector_USB:USB_Micro-B_Wuerth_614105150721_Vertical"
+		(property "Footprint" "xESC2:USB_Micro"
 			(at 57.15 44.45 0)
 			(effects
@@
 			)
 		)
-		(property "JLC" "C668588"
+		(property "JLC" "C145795"
 			(at 60.96 43.18 0)
 			(effects
