File: PCB/MCU.kicad_sch (KiCad schematic)
At the start: 14 parts, among them U4 STM32F405RGTx, Y1 Crystal_GND24

Commit message: Updated USB plug, Updated Part Numbers
Parts:
- C35, C36, C38, C39: JLC C49217 -> C377773; LCSC C49217 -> C377773
Changed lines of the file:
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@@
 			)
 		)
-		(property "JLC" "C49217"
+		(property "JLC" "C377773"
 			(at 53.34 60.96 0)
 			(effects
@@
 			)
 		)
-		(property "LCSC" "C49217"
+		(property "LCSC" "C377773"
 			(at 53.34 60.96 0)
 			(effects
@@
 			)
 		)
-		(property "JLC" "C49217"
+		(property "JLC" "C377773"
 			(at 44.45 58.42 0)
 			(effects
@@
 			)
 		)
-		(property "LCSC" "C49217"
+		(property "LCSC" "C377773"
 			(at 44.45 58.42 0)
 			(effects
@@
 			)
 		)
-		(property "JLC" "C49217"
+		(property "JLC" "C377773"
 			(at 161.29 29.21 0)
 			(effects
@@
 			)
 		)
-		(property "LCSC" "C49217"
+		(property "LCSC" "C377773"
 			(at 161.29 29.21 0)
 			(effects
@@
 			)
 		)
-		(property "JLC" "C49217"
+		(property "JLC" "C377773"
 			(at 153.67 29.21 0)
 			(effects
@@
 			)
 		)
-		(property "LCSC" "C49217"
+		(property "LCSC" "C377773"
 			(at 153.67 29.21 0)
 			(effects

Commit message: Updated Y1 Part Number
Parts:
- Y1: JLC C2442665 -> C2682775; LCSC C2442665 -> C2682775
Changed lines of the file:
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@@
 			)
 		)
-		(property "JLC" "C2442665"
+		(property "JLC" "C2682775"
 			(at 25.4 77.47 0)
 			(effects
@@
 			)
 		)
-		(property "LCSC" "C2442665"
+		(property "LCSC" "C2682775"
 			(at 25.4 77.47 0)
 			(effects
